File: wingbeat_detector/assembly.kicad_sch (KiCad schematic)
At the start: 8 parts

Commit message: Finished layout for v3.0
Other:
- company: Howard Hughes Medical Institute -> Peter Polidoro
Changed lines of the file:
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@@
   (title_block
     (title "wingbeat_detector")
-    (date "2023-03-22")
+    (date "2023-03-23")
     (rev "3.0")
-    (company "Howard Hughes Medical Institute")
+    (company "Peter Polidoro")
   )
   (wire (pts (xy 118.11 93.98) (xy 118.11 96.52))

Commit message: Update bom
Parts:
- H1, H2, H3, H4: now left out of the parts list
Changed lines of the file:
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@@
   )
   (symbol (lib_id "Janelia:MOUNTING_HOLE_2") (at 179.07 93.98 0) (unit 1)
-    (in_bom yes) (on_board yes) (dnp no) (fields_autoplaced)
-    (property "Reference" "H4" (at 179.07 87.122 0)
-      (effects (font (size 1.27 1.27)))
+    (in_bom no) (on_board yes) (dnp no) (fields_autoplaced)
+    (property "Reference" "H4" (at 181.61 91.313 0)
+      (effects (font (size 1.27 1.27)) (justify left))
     )
-    (property "Value" "MOUNTING_HOLE_2" (at 179.07 88.9 0)
-      (effects (font (size 1.27 1.27)))
+    (property "Value" "MOUNTING_HOLE_2" (at 179.07 101.6 0)
+      (effects (font (size 1.27 1.27)) hide)
     )
-    (property "Footprint" "Janelia:MOUNTING_HOLE_2" (at 184.15 93.98 0)
+    (property "Footprint" "Janelia:MOUNTING_HOLE_2" (at 179.07 104.14 0)
       (effects (font (size 1.27 1.27)) hide)
     )
     (property "Datasheet" "" (at 184.15 93.98 0)
+      (effects (font (size 1.27 1.27)) hide)
+    )
+    (property "Sim.Enable" "0" (at 179.07 93.98 0)
       (effects (font (size 1.27 1.27)) hide)
     )
@@
   )
   (symbol (lib_id "Janelia:MOUNTING_HOLE_2") (at 118.11 93.98 0) (unit 1)
-    (in_bom yes) (on_board yes) (dnp no) (fields_autoplaced)
-    (property "Reference" "H1" (at 118.11 87.122 0)
-      (effects (font (size 1.27 1.27)))
+    (in_bom no) (on_board yes) (dnp no) (fields_autoplaced)
+    (property "Reference" "H1" (at 120.65 91.313 0)
+      (effects (font (size 1.27 1.27)) (justify left))
     )
-    (property "Value" "MOUNTING_HOLE_2" (at 118.11 88.9 0)
-      (effects (font (size 1.27 1.27)))
+    (property "Value" "MOUNTING_HOLE_2" (at 118.11 101.6 0)
+      (effects (font (size 1.27 1.27)) hide)
     )
-    (property "Footprint" "Janelia:MOUNTING_HOLE_2" (at 123.19 93.98 0)
+    (property "Footprint" "Janelia:MOUNTING_HOLE_2" (at 118.11 104.14 0)
       (effects (font (size 1.27 1.27)) hide)
     )
     (property "Datasheet" "" (at 123.19 93.98 0)
+      (effects (font (size 1.27 1.27)) hide)
+    )
+    (property "Sim.Enable" "0" (at 118.11 93.98 0)
       (effects (font (size 1.27 1.27)) hide)
     )
@@
   )
   (symbol (lib_id "Janelia:MOUNTING_HOLE_2") (at 138.43 93.98 0) (unit 1)
-    (in_bom yes) (on_board yes) (dnp no) (fields_autoplaced)
-    (property "Reference" "H2" (at 138.43 87.122 0)
-      (effects (font (size 1.27 1.27)))
+    (in_bom no) (on_board yes) (dnp no) (fields_autoplaced)
+    (property "Reference" "H2" (at 140.97 91.313 0)
+      (effects (font (size 1.27 1.27)) (justify left))
     )
-    (property "Value" "MOUNTING_HOLE_2" (at 138.43 88.9 0)
-      (effects (font (size 1.27 1.27)))
+    (property "Value" "MOUNTING_HOLE_2" (at 138.43 101.6 0)
+      (effects (font (size 1.27 1.27)) hide)
     )
-    (property "Footprint" "Janelia:MOUNTING_HOLE_2" (at 143.51 93.98 0)
+    (property "Footprint" "Janelia:MOUNTING_HOLE_2" (at 138.43 104.14 0)
       (effects (font (size 1.27 1.27)) hide)
     )
     (property "Datasheet" "" (at 143.51 93.98 0)
+      (effects (font (size 1.27 1.27)) hide)
+    )
+    (property "Sim.Enable" "0" (at 138.43 93.98 0)
       (effects (font (size 1.27 1.27)) hide)
     )
@@
   )
   (symbol (lib_id "Janelia:MOUNTING_HOLE_2") (at 158.75 93.98 0) (unit 1)
-    (in_bom yes) (on_board yes) (dnp no) (fields_autoplaced)
-    (property "Reference" "H3" (at 158.75 87.122 0)
-      (effects (font (size 1.27 1.27)))
+    (in_bom no) (on_board yes) (dnp no) (fields_autoplaced)
+    (property "Reference" "H3" (at 161.29 91.313 0)
+      (effects (font (size 1.27 1.27)) (justify left))
     )
-    (property "Value" "MOUNTING_HOLE_2" (at 158.75 88.9 0)
-      (effects (font (size 1.27 1.27)))
+    (property "Value" "MOUNTING_HOLE_2" (at 158.75 101.6 0)
+      (effects (font (size 1.27 1.27)) hide)
     )
-    (property "Footprint" "Janelia:MOUNTING_HOLE_2" (at 163.83 93.98 0)
+    (property "Footprint" "Janelia:MOUNTING_HOLE_2" (at 158.75 104.14 0)
       (effects (font (size 1.27 1.27)) hide)
     )
@@
       (effects (font (size 1.27 1.27)) hide)
     )
+    (property "Sim.Enable" "0" (at 158.75 93.98 0)
+      (effects (font (size 1.27 1.27)) hide)
+    )
