File: wingbeat_detector/filter.kicad_sch (KiCad schematic)
At the start: 17 parts, among them J2 UMC_JACK_SMD, U2 UAF42_SMA

Commit message: Update images and documentation
Parts:
- R14: value GAIN1 -> 150k
Other:
- note added: "Vout/Vin = FILTER GAIN = Ra/Rb + 1 Low Gain: 5k/249 + 1 = 21 High Gain: 500k/249 + 1 = 2009"
- note removed: "Vout/Vin = GAIN1 = Ra/Rb + 1 Low Gain: 5k/249 + 1 = 21 High Gain: 500k/249 + 1 = 2009"
Changed lines of the file:
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@@
   (title_block
     (title "wingbeat_detector")
-    (date "2023-12-13")
+    (date "2023-12-14")
     (rev "4.0")
     (company "Peter Polidoro")
@@
     (effects (font (size 1.27 1.27)) (justify left bottom))
   )
-  (text "Vout/Vin = GAIN1 = Ra/Rb + 1\nLow Gain: 5k/249 + 1 = 21\nHigh Gain: 500k/249 + 1 = 2009 "
+  (text "Vout/Vin = FILTER GAIN = Ra/Rb + 1\nLow Gain: 5k/249 + 1 = 21\nHigh Gain: 500k/249 + 1 = 2009 "
     (at 161.29 49.53 0)
     (effects (font (size 1.27 1.27)) (justify left bottom))
@@
       (effects (font (size 1.016 1.016)))
     )
-    (property "Value" "GAIN1" (at 176.53 53.34 90) (do_not_autoplace)
-      (effects (font (size 0.762 0.762)))
-    )
+    (property "Value" "150k" (at 176.53 53.34 90) (do_not_autoplace)
+      (effects (font (size 0.762 0.762)))
+    )

Commit message: Change columns for manufacturer and manufacturer part number
Parts:
- C6, C7, C8, C9: MFN (none) -> Yageo; MPN (none) -> CC0402ZRY5V8BB104; Manufacturer Yageo -> (none); Manufacturer Part Number CC0402ZRY5V8BB104 -> (none)
- J2: MFN (none) -> Amphenol RF; MPN (none) -> A-1JB; Manufacturer Amphenol RF -> (none); Manufacturer Part Number A-1JB -> (none)
- R1, R3, R6, R8: MFN (none) -> Panasonic Electronic Components; MPN (none) -> ERJ-2RKF4992X; Manufacturer Panasonic Electronic Components -> (none); Manufacturer Part Number ERJ-2RKF4992X -> (none)
- R14: MFN (none) -> Panasonic Electronic Components; MPN (none) -> ERA-8AEB154V; Manufacturer Panasonic Electronic Components -> (none); Manufacturer Part Number ERA-8AEB154V -> (none)
- R2, R4: MFN (none) -> Panasonic Electronic Components; MPN (none) -> ERJ-2RKF6812X; Manufacturer Panasonic Electronic Components -> (none); Manufacturer Part Number ERJ-2RKF6812X -> (none)
- R5, R7: MFN (none) -> Vishay Dale; MPN (none) -> CRCW06033M65FKEA; Manufacturer Vishay Dale -> (none); Manufacturer Part Number CRCW06033M65FKEA -> (none)
- R9: MFN (none) -> Panasonic Electronic Components; MPN (none) -> ERJ-2RKF2490X; Manufacturer Panasonic Electronic Components -> (none); Manufacturer Part Number ERJ-2RKF2490X -> (none)
- U2: MFN (none) -> Texas Instruments; MPN (none) -> UAF42AU; Manufacturer Texas Instruments -> (none); Manufacturer Part Number UAF42AU -> (none)
Changed lines of the file:
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@@
       (effects (font (size 1.524 1.524)) hide)
     )
-    (property "Manufacturer" "Texas Instruments" (at 129.54 152.4 0)
-      (effects (font (size 1.27 1.27)) hide)
-    )
-    (property "Manufacturer Part Number" "UAF42AU" (at 129.54 152.4 0)
+    (property "MFN" "Texas Instruments" (at 129.54 152.4 0)
+      (effects (font (size 1.27 1.27)) hide)
+    )
+    (property "MPN" "UAF42AU" (at 129.54 152.4 0)
       (effects (font (size 1.27 1.27)) hide)
     )
@@
       (effects (font (size 1.524 1.524)) hide)
     )
-    (property "Manufacturer" "Texas Instruments" (at 129.54 76.2 0)
-      (effects (font (size 1.27 1.27)) hide)
-    )
-    (property "Manufacturer Part Number" "UAF42AU" (at 129.54 76.2 0)
+    (property "MFN" "Texas Instruments" (at 129.54 76.2 0)
+      (effects (font (size 1.27 1.27)) hide)
+    )
+    (property "MPN" "UAF42AU" (at 129.54 76.2 0)
       (effects (font (size 1.27 1.27)) hide)
     )
@@
       (effects (font (size 1.27 1.27)) hide)
     )
-    (property "Manufacturer" "Panasonic Electronic Components" (at 167.64 62.23 0)
-      (effects (font (size 1.27 1.27)) hide)
-    )
-    (property "Manufacturer Part Number" "ERJ-2RKF2490X" (at 167.64 62.23 0)
+    (property "MFN" "Panasonic Electronic Components" (at 167.64 62.23 0)
+      (effects (font (size 1.27 1.27)) hide)
+    )
+    (property "MPN" "ERJ-2RKF2490X" (at 167.64 62.23 0)
       (effects (font (size 1.27 1.27)) hide)
     )
@@
       (effects (font (size 1.27 1.27)) hide)
     )
-    (property "Manufacturer" "Panasonic Electronic Components" (at 92.71 146.05 0)
-      (effects (font (size 1.27 1.27)) hide)
-    )
-    (property "Manufacturer Part Number" "ERJ-2RKF4992X" (at 92.71 146.05 0)
+    (property "MFN" "Panasonic Electronic Components" (at 92.71 146.05 0)
+      (effects (font (size 1.27 1.27)) hide)
+    )
+    (property "MPN" "ERJ-2RKF4992X" (at 92.71 146.05 0)
       (effects (font (size 1.27 1.27)) hide)
     )
@@
       (effects (font (size 1.27 1.27)) hide)
     )
-    (property "Manufacturer" "Amphenol RF" (at 231.14 93.98 0)
-      (effects (font (size 1.27 1.27)) hide)
-    )
-    (property "Manufacturer Part Number" "A-1JB" (at 231.14 119.38 0)
+    (property "MFN" "Amphenol RF" (at 231.14 93.98 0)
+      (effects (font (size 1.27 1.27)) hide)
+    )
+    (property "MPN" "A-1JB" (at 231.14 119.38 0)
       (effects (font (size 1.27 1.27)) hide)
     )
@@
       (effects (font (size 1.27 1.27)) hide)
     )
-    (property "Manufacturer" "Vishay Dale" (at 114.3 50.8 0)
-      (effects (font (size 1.27 1.27)) hide)
-    )
-    (property "Manufacturer Part Number" "CRCW06033M65FKEA" (at 114.3 50.8 0)
+    (property "MFN" "Vishay Dale" (at 114.3 50.8 0)
+      (effects (font (size 1.27 1.27)) hide)
+    )
+    (property "MPN" "CRCW06033M65FKEA" (at 114.3 50.8 0)
       (effects (font (size 1.27 1.27)) hide)
     )
@@
       (effects (font (size 1.27 1.27)) hide)
     )
-    (property "Manufacturer" "Vishay Dale" (at 132.08 50.8 0)
-      (effects (font (size 1.27 1.27)) hide)
-    )
-    (property "Manufacturer Part Number" "CRCW06033M65FKEA" (at 132.08 50.8 0)
+    (property "MFN" "Vishay Dale" (at 132.08 50.8 0)
+      (effects (font (size 1.27 1.27)) hide)
+    )
+    (property "MPN" "CRCW06033M65FKEA" (at 132.08 50.8 0)
       (effects (font (size 1.27 1.27)) hide)
     )
@@
       (effects (font (size 1.27 1.27)) hide)
     )
-    (property "Manufacturer" "Yageo" (at 80.01 167.64 0)
-      (effects (font (size 1.27 1.27)) hide)
-    )
-    (property "Manufacturer Part Number" "CC0402ZRY5V8BB104" (at 80.01 167.64 0)
+    (property "MFN" "Yageo" (at 80.01 167.64 0)
+      (effects (font (size 1.27 1.27)) hide)
+    )
+    (property "MPN" "CC0402ZRY5V8BB104" (at 80.01 167.64 0)
       (effects (font (size 1.27 1.27)) hide)
     )
@@
       (effects (font (size 1.27 1.27)) hide)
     )
-    (property "Manufacturer" "Panasonic Electronic Components" (at 92.71 166.37 0)
-      (effects (font (size 1.27 1.27)) hide)
-    )
-    (property "Manufacturer Part Number" "ERJ-2RKF6812X" (at 92.71 166.37 0)
+    (property "MFN" "Panasonic Electronic Components" (at 92.71 166.37 0)
+      (effects (font (size 1.27 1.27)) hide)
+    )
+    (property "MPN" "ERJ-2RKF6812X" (at 92.71 166.37 0)
       (effects (font (size 1.27 1.27)) hide)
     )
@@
       (effects (font (size 1.27 1.27)) hide)
     )
-    (property "Manufacturer" "Yageo" (at 80.01 91.44 0)
-      (effects (font (size 1.27 1.27)) hide)
-    )
-    (property "Manufacturer Part Number" "CC0402ZRY5V8BB104" (at 80.01 91.44 0)
+    (property "MFN" "Yageo" (at 80.01 91.44 0)
+      (effects (font (size 1.27 1.27)) hide)
+    )
+    (property "MPN" "CC0402ZRY5V8BB104" (at 80.01 91.44 0)
       (effects (font (size 1.27 1.27)) hide)
     )
@@
       (effects (font (size 1.27 1.27)) hide)
     )
-    (property "Manufacturer" "Panasonic Electronic Components" (at 92.71 69.85 0)
-      (effects (font (size 1.27 1.27)) hide)
-    )
-    (property "Manufacturer Part Number" "ERJ-2RKF4992X" (at 92.71 69.85 0)
+    (property "MFN" "Panasonic Electronic Components" (at 92.71 69.85 0)
+      (effects (font (size 1.27 1.27)) hide)
+    )
+    (property "MPN" "ERJ-2RKF4992X" (at 92.71 69.85 0)
       (effects (font (size 1.27 1.27)) hide)
     )
@@
       (effects (font (size 1.27 1.27)) hide)
     )
-    (property "Manufacturer" "Yageo" (at 72.39 167.64 0)
-      (effects (font (size 1.27 1.27)) hide)
-    )
-    (property "Manufacturer Part Number" "CC0402ZRY5V8BB104" (at 72.39 167.64 0)
+    (property "MFN" "Yageo" (at 72.39 167.64 0)
+      (effects (font (size 1.27 1.27)) hide)
+    )
+    (property "MPN" "CC0402ZRY5V8BB104" (at 72.39 167.64 0)
       (effects (font (size 1.27 1.27)) hide)
     )
@@
       (effects (font (size 1.27 1.27)) hide)
     )
-    (property "Manufacturer" "Panasonic Electronic Components" (at 92.71 90.17 0)
-      (effects (font (size 1.27 1.27)) hide)
-    )
-    (property "Manufacturer Part Number" "ERJ-2RKF6812X" (at 92.71 90.17 0)
+    (property "MFN" "Panasonic Electronic Components" (at 92.71 90.17 0)
+      (effects (font (size 1.27 1.27)) hide)
+    )
+    (property "MPN" "ERJ-2RKF6812X" (at 92.71 90.17 0)
       (effects (font (size 1.27 1.27)) hide)
     )
@@
       (effects (font (size 1.27 1.27)) hide)
     )
-    (property "Manufacturer" "Panasonic Electronic Components" (at 176.53 53.34 0)
-      (effects (font (size 1.27 1.27)) hide)
-    )
-    (property "Manufacturer Part Number" "ERA-8AEB154V" (at 176.53 53.34 0)
+    (property "MFN" "Panasonic Electronic Components" (at 176.53 53.34 0)
+      (effects (font (size 1.27 1.27)) hide)
+    )
+    (property "MPN" "ERA-8AEB154V" (at 176.53 53.34 0)
       (effects (font (size 1.27 1.27)) hide)
     )
@@
       (effects (font (size 1.27 1.27)) hide)
     )
-    (property "Manufacturer" "Panasonic Electronic Components" (at 132.08 127 0)
-      (effects (font (size 1.27 1.27)) hide)
-    )
-    (property "Manufacturer Part Number" "ERJ-2RKF4992X" (at 132.08 127 0)
+    (property "MFN" "Panasonic Electronic Components" (at 132.08 127 0)
+      (effects (font (size 1.27 1.27)) hide)
+    )
+    (property "MPN" "ERJ-2RKF4992X" (at 132.08 127 0)
       (effects (font (size 1.27 1.27)) hide)
     )
@@
       (effects (font (size 1.27 1.27)) hide)
     )
-    (property "Manufacturer" "Yageo" (at 72.39 91.44 0)
-      (effects (font (size 1.27 1.27)) hide)
-    )
-    (property "Manufacturer Part Number" "CC0402ZRY5V8BB104" (at 72.39 91.44 0)
+    (property "MFN" "Yageo" (at 72.39 91.44 0)
+      (effects (font (size 1.27 1.27)) hide)
+    )
+    (property "MPN" "CC0402ZRY5V8BB104" (at 72.39 91.44 0)
       (effects (font (size 1.27 1.27)) hide)
     )
@@
       (effects (font (size 1.27 1.27)) hide)
     )
-    (property "Manufacturer" "Panasonic Electronic Components" (at 114.3 127 0)
-      (effects (font (size 1.27 1.27)) hide)
-    )
-    (property "Manufacturer Part Number" "ERJ-2RKF4992X" (at 114.3 127 0)
-      (effects (font (size 1.27 1.27)) hide)
-    )
+    (property "MFN" "Panasonic Electronic Components" (at 114.3 127 0)
+      (effects (font (size 1.27 1.27)) hide)
+    )
+    (property "MPN" "ERJ-2RKF4992X" (at 114.3 127 0)
+      (effects (font (size 1.27 1.27)) hide)
+    )
