File: wingbeat_detector/photodiode.kicad_sch (KiCad schematic)
At the start: 6 parts, among them J2 UMC_JACK_SMD, U4 OPA381

Commit message: Update images and documentation
Other:
- note added: "DIODE GAIN MIN: R = (5V - 0.6V)/90uA = 48.8k MAX: R = (5V - 0.6V)/0.8uA = 5.5M"
- note removed: "GAIN0 MIN: R = (5V - 0.6V)/90uA = 48.8k GAIN0 MAX: R = (5V - 0.6V)/0.8uA = 5.5M"
Changed lines of the file:
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@@
   (title_block
     (title "wingbeat_detector")
-    (date "2023-12-13")
+    (date "2023-12-14")
     (rev "4.0")
     (company "Peter Polidoro")
@@
     (stroke (width 0) (type default))
   )
-  (text "GAIN0 MIN: R = (5V - 0.6V)/90uA = 48.8k\nGAIN0 MAX: R = (5V - 0.6V)/0.8uA = 5.5M"
-    (at 149.86 66.04 0)
+  (text "DIODE GAIN\nMIN: R = (5V - 0.6V)/90uA = 48.8k\nMAX: R = (5V - 0.6V)/0.8uA = 5.5M"
+    (at 149.86 67.31 0)
     (effects (font (size 1.27 1.27)) (justify left bottom))
   )

Commit message: Change columns for manufacturer and manufacturer part number
Parts:
- C10: MFN (none) -> Samsung Electro-Mechanics; MPN (none) -> CL05A105KL5NRNC; Manufacturer Samsung Electro-Mechanics -> (none); Manufacturer Part Number CL05A105KL5NRNC -> (none)
- C11: MFN (none) -> KEMET; MPN (none) -> C0402C300J5GACAUTO; Manufacturer KEMET -> (none); Manufacturer Part Number C0402C300J5GACAUTO -> (none)
- D1: MFN (none) -> American Bright Optoelectronics Corporation; MPN (none) -> BPD-BQDA38V-FZ04; Manufacturer American Bright Optoelectronics Corporation -> (none); Manufacturer Part Number BPD-BQDA38V-FZ04 -> (none)
- J2: MFN (none) -> Amphenol RF; MPN (none) -> A-1JB; Manufacturer Amphenol RF -> (none); Manufacturer Part Number A-1JB -> (none)
- R11: MFN (none) -> Panasonic Electronic Components; MPN (none) -> ERJ-PM8F2004V; Manufacturer Panasonic Electronic Components -> (none); Manufacturer Part Number ERJ-PM8F2004V -> (none)
- U4: MFN (none) -> Texas Instruments; MPN (none) -> OPA381AIDRBT; Manufacturer Texas Instruments -> (none); Manufacturer Part Number OPA381AIDRBT -> (none)
Changed lines of the file:
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@@
       (effects (font (size 1.27 1.27)) hide)
     )
-    (property "Manufacturer" "Panasonic Electronic Components" (at 138.43 64.77 0)
-      (effects (font (size 1.27 1.27)) hide)
-    )
-    (property "Manufacturer Part Number" "ERJ-PM8F2004V" (at 138.43 64.77 0)
+    (property "MFN" "Panasonic Electronic Components" (at 138.43 64.77 0)
+      (effects (font (size 1.27 1.27)) hide)
+    )
+    (property "MPN" "ERJ-PM8F2004V" (at 138.43 64.77 0)
       (effects (font (size 1.27 1.27)) hide)
     )
@@
       (effects (font (size 1.27 1.27)) hide)
     )
-    (property "Manufacturer" "Texas Instruments" (at 138.43 57.15 0)
-      (effects (font (size 1.27 1.27)) hide)
-    )
-    (property "Manufacturer Part Number" "OPA381AIDRBT" (at 138.43 52.07 0)
+    (property "MFN" "Texas Instruments" (at 138.43 57.15 0)
+      (effects (font (size 1.27 1.27)) hide)
+    )
+    (property "MPN" "OPA381AIDRBT" (at 138.43 52.07 0)
       (effects (font (size 1.27 1.27)) hide)
     )
@@
       (effects (font (size 1.27 1.27)) hide)
     )
-    (property "Manufacturer" "Amphenol RF" (at 208.28 96.52 0)
-      (effects (font (size 1.27 1.27)) hide)
-    )
-    (property "Manufacturer Part Number" "A-1JB" (at 208.28 121.92 0)
+    (property "MFN" "Amphenol RF" (at 208.28 96.52 0)
+      (effects (font (size 1.27 1.27)) hide)
+    )
+    (property "MPN" "A-1JB" (at 208.28 121.92 0)
       (effects (font (size 1.27 1.27)) hide)
     )
@@
       (effects (font (size 1.27 1.27)) hide)
     )
-    (property "Manufacturer" "American Bright Optoelectronics Corporation" (at 129.54 90.17 0)
-      (effects (font (size 1.27 1.27)) hide)
-    )
-    (property "Manufacturer Part Number" "BPD-BQDA38V-FZ04" (at 121.92 90.17 0)
+    (property "MFN" "American Bright Optoelectronics Corporation" (at 129.54 90.17 0)
+      (effects (font (size 1.27 1.27)) hide)
+    )
+    (property "MPN" "BPD-BQDA38V-FZ04" (at 121.92 90.17 0)
       (effects (font (size 1.27 1.27)) hide)
     )
@@
       (effects (font (size 1.27 1.27)) hide)
     )
-    (property "Manufacturer" "Samsung Electro-Mechanics" (at 81.28 88.9 0)
-      (effects (font (size 1.27 1.27)) hide)
-    )
-    (property "Manufacturer Part Number" "CL05A105KL5NRNC" (at 81.28 88.9 0)
+    (property "MFN" "Samsung Electro-Mechanics" (at 81.28 88.9 0)
+      (effects (font (size 1.27 1.27)) hide)
+    )
+    (property "MPN" "CL05A105KL5NRNC" (at 81.28 88.9 0)
       (effects (font (size 1.27 1.27)) hide)
     )
@@
       (effects (font (size 1.27 1.27)) hide)
     )
-    (property "Manufacturer" "KEMET" (at 138.43 54.61 0)
-      (effects (font (size 1.27 1.27)) hide)
-    )
-    (property "Manufacturer Part Number" "C0402C300J5GACAUTO" (at 138.43 54.61 0)
-      (effects (font (size 1.27 1.27)) hide)
-    )
+    (property "MFN" "KEMET" (at 138.43 54.61 0)
+      (effects (font (size 1.27 1.27)) hide)
+    )
+    (property "MPN" "C0402C300J5GACAUTO" (at 138.43 54.61 0)
+      (effects (font (size 1.27 1.27)) hide)
+    )
